Commit message: created rviz file and launched it

File: src/my_bot_description/urdf/my_bot.urdf.xacro (robot description, xacro)
@@ -43,29 +43,28 @@
         <axis xyz="0 1 0"/>
     </joint>
-    <link name="castor_front_link">
+    <link name="caster_front_link">
         <visual>
+            <origin rpy="0 0 0" xyz="0 0 0"/>
             <geometry>
-                <origin rpy="0 0 0" xyz="0 0 0"/>
-                <mesh filename="package://my_bot_description/meshes/castor_front_link.stl"/>
+                <mesh filename="package://my_bot_description/meshes/caster_front_link.stl"/>
             </geometry>
         </visual>
     </link>
-    <joint name="castor_front_joint" type="fixed">
+    <joint name="caster_front_joint" type="fixed">
         <parent link="base_link"/>
-        <child link="castor_front_link"/>
+        <child link="caster_front_link"/>
         <origin rpy="0 0 0" xyz="0.04755 0 -0.0275"/>
     </joint>
-    <link name="castor_rear_link">
+    <link name="caster_rear_link">
         <visual>
+            <origin rpy="0 0 0" xyz="0 0 0"/>
             <geometry>
-                <origin rpy="0 0 0" xyz="0 0 0"/>
-                <!mesh filename="package://my_bot_description/meshes/castor_rear_link.stl"/>
-                <box size="0.02 0.02 0.02"/>
+                <mesh filename="package://my_bot_description/meshes/caster_rear_link.stl"/>
             </geometry>
         </visual>
     </link>
-    <joint name="castor_rear_joint" type="fixed">
+    <joint name="caster_rear_joint" type="fixed">
         <parent link="base_link"/>
-        <child link="castor_rear_link"/>
+        <child link="caster_rear_link"/>
         <origin rpy="0 0 0" xyz="-0.04755 0 -0.0275"/>
     </joint>

Commit message: added inertial and collision tags with gazebo launch files

File: src/my_bot_description/urdf/my_bot.urdf.xacro (robot description, xacro)
@@ -1,4 +1,5 @@
 <?xml version="1.0"?>
 <robot xmlns:xacro="http://www.ros.org/wiki/xacro" name="my_bot">
+    <xacro:include filename="package://my_bot_description/urdf/my_bot_gazebo.xacro"/>
     <link name="base_footprint"/>
     <link name="base_link">
@@ -9,4 +10,17 @@
             </geometry>
         </visual>
+        <collision>
+            <origin rpy="0 0 0" xyz="0 0 0"/>
+            <geometry>
+                <mesh filename="package://my_bot_description/meshes/base_link.stl"/>
+            </geometry>
+        </collision>
+        <inertial>
+            <origin xyz="0 0 0.04" rpy="0.0 0.25 0.3"/>
+            <mass value="8.2573504e-01"/>
+            <inertia ixx="2.2124416e-02" ixy="-1.2294101e-04" ixz="3.4938785e-04"
+               iyy="2.1193702e-02" iyz="-5.0120904e-05"
+               izz="2.0064271e-02" />
+        </inertial>
     </link>
     <joint name="base_joint" type="fixed">
@@ -22,4 +36,17 @@
             </geometry>
         </visual>
+        <collision>
+            <origin rpy="1.57 0 0" xyz="0 -0.015 0"/>
+             <geometry>
+                <sphere radius="0.033"/>
+            </geometry>
+        </collision>
+        <inertial>
+            <origin xyz="0 -0.014 0" rpy="0 0 0" />
+            <mass value="0.0530086090966721" />
+            <inertia ixx="1.88176298336665E-05" ixy="-4.8444933029987E-10" ixz="1.88163708851143E-08"
+                    iyy="3.11510738647764E-05" iyz="-6.93560663069607E-11"
+                    izz="1.8801969558182E-05" />
+        </inertial>
     </link>
     <joint name="wheel_right_joint" type="continuous">
@@ -36,4 +63,17 @@
             </geometry>
         </visual>
+        <collision>
+            <origin rpy="1.57 0 0" xyz="0 0.015 0"/>
+             <geometry>
+                <sphere radius="0.033"/>
+            </geometry>
+        </collision>
+        <inertial>
+            <origin xyz="0 0.014 0" rpy="0 0 0" />
+            <mass value="0.0530086043217644" />
+            <inertia ixx="1.8792911368909E-05"  ixy="3.31256392204584E-10" ixz="-1.14082001662767E-08"
+                    iyy="3.11510738759073E-05" iyz="-3.60499245082192E-10"
+                    izz="1.88266886146847E-05" />
+        </inertial>
     </link>
     <joint name="wheel_left_joint" type="continuous">
@@ -50,4 +90,17 @@
             </geometry>
         </visual>
+        <collision>
+            <origin rpy="0 0 0" xyz="0 0 0"/>
+            <geometry>
+                <sphere radius="0.005"/>
+            </geometry>
+        </collision>
+        <inertial>
+            <origin xyz="3.89968128948481E-07 2.40073004698083E-07 0.00219173397061506" rpy="0 0 0" />
+            <mass value="1.44379265037903E-06" />
+            <inertia ixx="7.23075276010246E-11" ixy="-6.10956883467859E-16" ixz="2.22849693525031E-15"
+                    iyy="3.8713793085917E-11"  iyz="2.93909858781952E-15"
+                    izz="1.00967486676306E-10" />
+        </inertial>
     </link>
     <joint name="caster_front_joint" type="fixed">
@@ -63,4 +116,17 @@
             </geometry>
         </visual>
+        <collision>
+            <origin rpy="0 0 0" xyz="0 0 0"/>
+            <geometry>
+                <sphere radius="0.005"/>
+            </geometry>
+        </collision>
+        <inertial>
+            <origin xyz="3.8996812895542E-07 2.40073004698083E-07 0.00219173397061509" rpy="0 0 0" />
+            <mass value="1.44379265037902E-06" />
+            <inertia ixx="7.23075276010246E-11" ixy="-6.10956872363424E-16" ixz="2.22849693527207E-15"
+                    iyy="3.87137930859167E-11" iyz="2.939098587861E-15"
+                    izz="1.00967486676306E-10" />
+        </inertial>
     </link>
     <joint name="caster_rear_joint" type="fixed">
